Commit message: add update rate

File: rosbot_description/urdf/rosbot.xacro (robot description, xacro)
@@ -3,7 +3,9 @@
   xmlns:xacro="http://www.ros.org/wiki/xacro">
   <xacro:arg name="robot_namespace" default=""/>
+  <xacro:arg name="update_rate"     default="10" />
   <xacro:property name="cameraSize" value="0.05"/>
   <xacro:property name="cameraMass" value="0.1"/>
   <xacro:property name="namespace" value="$(arg robot_namespace)" />
+  <xacro:property name="update_rate" value="$(arg update_rate)" />
   <xacro:include filename="$(find rosbot_description)/urdf/rosbot.gazebo" />
   <xacro:include filename="$(find rosbot_description)/urdf/materials.xacro" />
